File: pcb/MotionSense.brd (EAGLE design)
At the start: 61.6 x 60.6 mm, 14 parts

Commit message: [UPDATE] PCB update v2
Parts:
- removed MODUL1: ARDUINO_NANO2, arduino_2012:ARDUINO_NANO2
- added ARDUINO-NANO: ARDUINO_NANO2, arduino_2012:ARDUINO_NANO2
- moved SENSORS 87.8 mm to (39.6, 39.9), turned to 90 degrees
- moved U$1 87.5 mm to (33.4, 58.8), turned to 270 degrees
- moved BAT-IN 85.2 mm to (29.0, 39.6), turned to 90 degrees
- moved ON/OFF 76.7 mm to (30.1, 20.3), turned to 180 degrees
- moved PUSH-FUNC 67.6 mm to (72.6, 20.6)
- moved R5 62.9 mm to (52.2, 42.1), turned to 90 degrees
- moved R3 50.1 mm to (56.2, 39.6), turned to 90 degrees
- moved LED1 37.0 mm to (27.3, 29.5), turned to 90 degrees
- moved LED 31.4 mm to (36.7, 29.5), turned to 90 degrees
- moved PUSH-START 7.30 mm to (72.6, 29.6), turned to 0 degrees
- moved R2 4.82 mm to (74.8, 57.1)
- moved R1 3.92 mm to (69.7, 57.3)
- moved HC-05 1.69 mm to (72.5, 54.5)
Connections:
- net 3V3: now also ARDUINO-NANO.J2.14; no longer MODUL1.J2.14
- net AREF: now also ARDUINO-NANO.J2.13; no longer MODUL1.J2.13
- net N$10: now also ARDUINO-NANO.J1.15; no longer MODUL1.J1.15
- net N$11: now also ARDUINO-NANO.J2.1; no longer MODUL1.J2.1
- net N$12: now also ARDUINO-NANO.J1.12; no longer MODUL1.J1.12
- net N$13: now also ARDUINO-NANO.J1.9; no longer MODUL1.J1.9
- net N$2: now also ARDUINO-NANO.J2.4; no longer MODUL1.J2.4
- net N$3: now also ARDUINO-NANO.J1.14; no longer MODUL1.J1.14
- net N$4: now also ARDUINO-NANO.J2.2; no longer MODUL1.J2.2
- net N$5: now also ARDUINO-NANO.J1.13; no longer MODUL1.J1.13
- net N$7: now also ARDUINO-NANO.J2.7; no longer MODUL1.J2.7
- net N$8: now also ARDUINO-NANO.J2.8; no longer MODUL1.J2.8
- net N$9: now also ARDUINO-NANO.J1.10; no longer MODUL1.J1.10
- net NEGATIVE: now also ARDUINO-NANO.J1.4; no longer MODUL1.J1.4
Routing:
- net N$11: track 0.00 -> 74.7 mm, vias 0 -> 2
- net N$2: track 22.7 -> 91.2 mm, vias 1 -> 0
- net N$4: track 28.4 -> 93.7 mm, vias 0 -> 1
- net N$8: track 0.00 -> 56.8 mm
- net N$7: track 0.00 -> 54.4 mm
- net NEGATIVE: track 0.00 -> 51.4 mm
- net N$12: track 0.00 -> 51.0 mm, vias 0 -> 1
- net N$14: track 0.00 -> 44.3 mm, vias 0 -> 1
- net POSITIVE: track 0.00 -> 38.9 mm
- net N$1: track 0.00 -> 37.3 mm, vias 0 -> 1
- net N$3: track 76.2 -> 56.1 mm, vias 1 -> 3
- net N$10: track 43.5 -> 31.1 mm
- net N$9: track 0.00 -> 10.8 mm
- net N$5: track 108.7 -> 99.2 mm
- net N$13: track 0.00 -> 5.68 mm
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Other:
- board size 61.6 x 60.6 mm -> 59.4 x 59.2 mm
- board text added: "/home/wanghley/Desktop/brazil-flag-min.bmp"
- board text added: "/home/wanghley/Desktop/cnpq3.bmp"
- board text added: "/home/wanghley/Desktop/ifb.bmp"
- board text added: "Arduino Nano"
- board text added: "Developed by Wanghley Soares Martins (@wanghley) Prof. Fabio Henrique M. Oliveira (@oliveirafhm)"
- board text added: "INERTIAL DATA COLLECTION DEVICE"
- board text added: "V2.0"
- board text removed: "CNPq"
- board text removed: "Designed and Prototyped by:"
- board text removed: "IFB"
- board text removed: "Motion Sense"
- board text removed: "V1.0"
- board text removed: "Wanghley Soares Martins Prof. Fábio Henrique"
